Commit message: 2f_driver

File: delto_description/urdf/delto_gripper_2f.urdf (robot description, URDF)
Before this commit: robot delto_3f_description, 3 links, 2 joints
Links:
- link TIP1: geometry collision mesh filename=package://delto_description/meshes/DG2F/TIP.stl; visual mesh filename=package://delto_description/meshes/DG2F/TIP.stl
- link TIP2: geometry collision mesh filename=package://delto_description/meshes/DG2F/TIP.stl; visual mesh filename=package://delto_description/meshes/DG2F/TIP.stl
- link delto_base_link: geometry collision mesh filename=package://delto_description/meshes/DG2F/delto_base_link.stl; visual mesh filename=package://delto_description/meshes/DG2F/delto_base_link.stl
Joints:
- removed joint JOINT1
- added joint Distance: type prismatic, parent delto_base_link, child TIP1, origin xyz=0 0 0.113 rpy=1.5708 0 -3.1345, axis -1 0 0, limit lower=0.0 upper=0.025 effort=1000.0 velocity=0.5
- joint JOINT2: mimic joint=JOINT1 multiplier=1 -> joint=Distance multiplier=1

Commit message: diplay fix

File: delto_description/urdf/delto_gripper_2f.urdf (robot description, URDF)
Before this commit: robot delto_description, 3 links, 2 joints
Links:
- link delto_base_link: geometry collision mesh filename=package://delto_description/meshes/DG2F/delto_base_link.stl; visual mesh filename=package://delto_description/meshes/DG2F/delto_base_link.dae
Joints:
- joint Distance: origin xyz=0 0 0.113 rpy=1.5708 0 -3.1345 -> xyz=0 0 0.113 rpy=1.5708 0 -3.141597
