Commit message: decription root

File: delto_3f_moveit/config/delto_gripper_3f.urdf.xacro (robot description, xacro)
@@ -3,5 +3,5 @@
     <xacro:arg name="initial_positions_file" default="initial_positions.yaml" />
     <!-- Import delto_gripper_3f urdf file -->
-    <xacro:include filename="$(find delto_3f_description)/urdf/delto_gripper_3f.urdf" />
+    <xacro:include filename="$(find delto_description)/urdf/delto_gripper_3f.urdf" />
     <!-- Import control_xacro -->
     <xacro:include filename="delto_gripper_3f.ros2_control.xacro" />

File: delto_description/urdf/delto_gripper_3f.urdf (robot description, URDF)
Before this commit: robot delto_gripper_3f, 16 links, 15 joints
Links:
- link F1_01: geometry collision mesh filename=package://delto_description/meshes/DG3F/link_01.stl; visual mesh filename=package://delto_description/meshes/DG3F/link_01.stl
- link F1_02: geometry collision mesh filename=package://delto_description/meshes/DG3F/link_02.stl; visual mesh filename=package://delto_description/meshes/DG3F/link_02.stl
- link F1_03: geometry collision mesh filename=package://delto_description/meshes/DG3F/link_03.stl; visual mesh filename=package://delto_description/meshes/DG3F/link_03.stl
- link F1_04: geometry collision mesh filename=package://delto_description/meshes/DG3F/link_04.stl; visual mesh filename=package://delto_description/meshes/DG3F/link_04.stl
- link F1_TIP: geometry collision mesh filename=package://delto_description/meshes/DG3F/link_tip_high.stl; visual mesh filename=package://delto_description/meshes/DG3F/link_tip_high.stl
- link F2_01: geometry collision mesh filename=package://delto_description/meshes/DG3F/link_01.stl; visual mesh filename=package://delto_description/meshes/DG3F/link_01.stl
- link F2_02: geometry collision mesh filename=package://delto_description/meshes/DG3F/link_02.stl; visual mesh filename=package://delto_description/meshes/DG3F/link_02.stl
- link F2_03: geometry collision mesh filename=package://delto_description/meshes/DG3F/link_03.stl; visual mesh filename=package://delto_description/meshes/DG3F/link_03.stl
- link F2_04: geometry collision mesh filename=package://delto_description/meshes/DG3F/link_04.stl; visual mesh filename=package://delto_description/meshes/DG3F/link_04.stl
- link F2_TIP: geometry collision mesh filename=package://delto_description/meshes/DG3F/link_tip_high.stl; visual mesh filename=package://delto_description/meshes/DG3F/link_tip_high.stl
- link F3_01: geometry collision mesh filename=package://delto_description/meshes/DG3F/link_01.stl; visual mesh filename=package://delto_description/meshes/DG3F/link_01.stl
- link F3_02: geometry collision mesh filename=package://delto_description/meshes/DG3F/link_02.stl; visual mesh filename=package://delto_description/meshes/DG3F/link_02.stl
- link F3_03: geometry collision mesh filename=package://delto_description/meshes/DG3F/link_03.stl; visual mesh filename=package://delto_description/meshes/DG3F/link_03.stl
- link F3_04: geometry collision mesh filename=package://delto_description/meshes/DG3F/link_04.stl; visual mesh filename=package://delto_description/meshes/DG3F/link_04.stl
- link F3_TIP: geometry collision mesh filename=package://delto_description/meshes/DG3F/link_tip_high.stl; visual mesh filename=package://delto_description/meshes/DG3F/link_tip_high.stl
- link delto_base_link: geometry collision mesh filename=package://delto_description/meshes/DG3F/delto_base_link.stl; visual mesh filename=package://delto_description/meshes/DG3F/delto_base_link.stl

File: delto_description/urdf/ur.urdf.xacro (robot description, xacro)
@@ -5,5 +5,5 @@
    <!-- import main macro -->
    <xacro:include filename="$(find ur_description)/urdf/ur_macro.xacro"/>
-   <xacro:include filename="$(find delto_3f_description)/urdf/delto_gripper_3f.urdf"/>
+   <xacro:include filename="$(find delto_description)/urdf/delto_gripper_3f.urdf"/>
    <!-- possible 'ur_type' values: ur3, ur3e, ur5, ur5e, ur10, ur10e, ur16e, ur20 -->
    <!-- the default value should raise an error in case this was called without defining the type -->

File: delto_description/urdf/ur_delto_gripper_3f.urdf (robot description, URDF)
Before this commit: robot delto_gripper_3f, 16 links, 16 joints
Links:
- link F1_01: geometry collision mesh filename=package://delto_description/meshes/link_01.stl; visual mesh filename=package://delto_description/meshes/link_01.stl
- link F1_02: geometry collision mesh filename=package://delto_description/meshes/link_02.stl; visual mesh filename=package://delto_description/meshes/link_02.stl
- link F1_03: geometry collision mesh filename=package://delto_description/meshes/link_03.stl; visual mesh filename=package://delto_description/meshes/link_03.stl
- link F1_04: geometry collision mesh filename=package://delto_description/meshes/link_04.stl; visual mesh filename=package://delto_description/meshes/link_04.stl
- link F1_TIP: geometry collision mesh filename=package://delto_description/meshes/link_tip_high.stl; visual mesh filename=package://delto_description/meshes/link_tip_high.stl
- link F2_01: geometry collision mesh filename=package://delto_description/meshes/link_01.stl; visual mesh filename=package://delto_description/meshes/link_01.stl
- link F2_02: geometry collision mesh filename=package://delto_description/meshes/link_02.stl; visual mesh filename=package://delto_description/meshes/link_02.stl
- link F2_03: geometry collision mesh filename=package://delto_description/meshes/link_03.stl; visual mesh filename=package://delto_description/meshes/link_03.stl
- link F2_04: geometry collision mesh filename=package://delto_description/meshes/link_04.stl; visual mesh filename=package://delto_description/meshes/link_04.stl
- link F2_TIP: geometry collision mesh filename=package://delto_description/meshes/link_tip_high.stl; visual mesh filename=package://delto_description/meshes/link_tip_high.stl
- link F3_01: geometry collision mesh filename=package://delto_description/meshes/link_01.stl; visual mesh filename=package://delto_description/meshes/link_01.stl
- link F3_02: geometry collision mesh filename=package://delto_description/meshes/link_02.stl; visual mesh filename=package://delto_description/meshes/link_02.stl
- link F3_03: geometry collision mesh filename=package://delto_description/meshes/link_03.stl; visual mesh filename=package://delto_description/meshes/link_03.stl
- link F3_04: geometry collision mesh filename=package://delto_description/meshes/link_04.stl; visual mesh filename=package://delto_description/meshes/link_04.stl
- link F3_TIP: geometry collision mesh filename=package://delto_description/meshes/link_tip_high.stl; visual mesh filename=package://delto_description/meshes/link_tip_high.stl
- link delto_base_link: geometry collision mesh filename=package://delto_description/meshes/delto_base_link.stl; visual mesh filename=package://delto_description/meshes/delto_base_link.stl
